File: HW/STM8_001_PWM_485/STM8_001_PWM_485.sch (KiCad schematic (older format))
At the start: 13 parts, among them J1 PWM1, J2 PWM2, J3 In1, J4 In2, J5 SWIM, SW1 Sw, U1 L78L05_SOT89, U2 STM8S001J3M, U3 SP3485EN

Commit message: PCB Docs Cleanup
Parts:
- U2: symbol BK_Common:STM8S001J3M -> STM8_001_PWM_485-rescue:STM8S001J3M-BK_Common
Other:
- moved on the sheet: C1, C2, C3, J1, J2, J3, J4, J5, R1, SW1, U1, U2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
